File: panda.kicad_pcb (KiCad board)
At the start: 4 copper layers, 122.9 x 136.7 mm, 262 parts, among them J1 Logic_Power_Switch, J10 PT_6, J11 4-Pin Load Cell, J12 5-Pin Load Cell, J13 Ignitor Screw Terminal, J14 Valve_1_PWR, J15 Valve_4_PWR, J16 Valve_2_PWR, J17 Valve_5_PWR, J18 Valve_3_PWR, J19 Valve_6_PWR, J2 XT60-M, J3 24V_Lockout_Key_Switch, J4 USB_C_Receptacle_USB2.0_16P, J5 PT_1, J6 PT_4, J7 PT_2, J8 PT_5, J9 PT_3, K1 G5Q-1A DC24, K2 G5Q-1 DC24, K3 G5Q-1 DC24, Q1 BSS138, Q10 BSS138, Q11 BSS138, Q2 BSS138, Q3 DMP6023LE-13, Q4 BSS138, Q5 BSS138, Q6 BSS138, Q7 BSS138, Q8 BSS138, Q9 BSS138, SW1 USAKRO UK-B0227-G4.3-B-250, SW2 USAKRO UK-B0227-G4.3-B-250, U1 LM3880-1AA, U10 ADS112C04, U11 ADS112C04, U12 INA187A1, U13 ADS112C04, U14 TLC555xPS, U2 LMR33630BDDA, U3 TPS78533QKVURQ1, U5 TPS78450QDBVRQ1, U6 LM66200DRLR, U7 ESP32-S3-WROOM-1U, U8 ADS112C04, U9 ADS112C04

Commit message: change connectors and more progress on pcb
Parts:
- removed J4: USB_C_Receptacle_USB2.0_16P, Connector_USB:USB_C_Receptacle_G-Switch_GT-USB-7010ASV
- added J20: 395934308, Library:CONN_SD-39543-002_NONE_08P_MOL, F.Cu at (149.7, 169.2)
- added J21: USB_C_Receptacle_USB2.0_16P, Connector_USB:USB_C_Receptacle_G-Switch_GT-USB-7051x, F.Cu at (108.7, 59.0)
- C3: footprint Capacitor_SMD:C_1206_3216Metric -> Capacitor_SMD:C_1812_4532Metric
- J1: footprint Connector_JST:JST_XH_B2B-XH-A_1x02_P2.50mm_Vertical -> Connector_Molex:Molex_KK-396_A-41791-0002_1x02_P3.96mm_Vertical
- J10: value PT_6 -> Conn_01x02; footprint Connector_JST:JST_XH_B2B-XH-A_1x02_P2.50mm_Vertical -> Connector_Molex:Molex_Micro-Fit_3.0_43650-0215_1x02_P3.00mm_Vertical
- J13: value Ignitor Screw Terminal -> Conn_02x01; footprint TerminalBlock_4Ucon:TerminalBlock_4Ucon_1x02_P3.50mm_Vertical -> Connector_Molex:Molex_Mini-Fit_Jr_5566-02A_2x01_P4.20mm_Vertical
- J14: value Valve_1_PWR -> Conn_01x02; footprint Connector_JST:JST_XH_B2B-XH-A_1x02_P2.50mm_Vertical -> Connector_Molex:Molex_Micro-Fit_3.0_43650-0215_1x02_P3.00mm_Vertical
- J15: value Valve_4_PWR -> Conn_01x02; footprint Connector_JST:JST_XH_B2B-XH-A_1x02_P2.50mm_Vertical -> Connector_Molex:Molex_Micro-Fit_3.0_43650-0215_1x02_P3.00mm_Vertical
- J16: value Valve_2_PWR -> Conn_01x02; footprint Connector_JST:JST_XH_B2B-XH-A_1x02_P2.50mm_Vertical -> Connector_Molex:Molex_Micro-Fit_3.0_43650-0215_1x02_P3.00mm_Vertical
- J17: value Valve_5_PWR -> Conn_01x02; footprint Connector_JST:JST_XH_B2B-XH-A_1x02_P2.50mm_Vertical -> Connector_Molex:Molex_Micro-Fit_3.0_43650-0215_1x02_P3.00mm_Vertical
- J18: value Valve_3_PWR -> Conn_01x02; footprint Connector_JST:JST_XH_B2B-XH-A_1x02_P2.50mm_Vertical -> Connector_Molex:Molex_Micro-Fit_3.0_43650-0215_1x02_P3.00mm_Vertical
- J19: value Valve_6_PWR -> Conn_02x01; footprint Connector_JST:JST_XH_B2B-XH-A_1x02_P2.50mm_Vertical -> Connector_Molex:Molex_Mini-Fit_Jr_5566-02A_2x01_P4.20mm_Vertical
- J2: value XT60-M -> Conn_01x02; footprint Connector_AMASS:AMASS_XT60PW-F_1x02_P7.20mm_Horizontal -> Connector_Molex:Molex_Micro-Fit_3.0_43650-0215_1x02_P3.00mm_Vertical
- J3: value 24V_Lockout_Key_Switch -> Conn_01x02; footprint Connector_JST:JST_XH_B2B-XH-A_1x02_P2.50mm_Vertical -> Connector_Molex:Molex_Micro-Fit_3.0_43650-0215_1x02_P3.00mm_Vertical
- J5: value PT_1 -> Conn_02x01; footprint Connector_JST:JST_XH_B2B-XH-A_1x02_P2.50mm_Vertical -> Connector_Molex:Molex_Mini-Fit_Jr_5566-02A_2x01_P4.20mm_Vertical
- J6: value PT_4 -> Conn_01x02; footprint Connector_JST:JST_XH_B2B-XH-A_1x02_P2.50mm_Vertical -> Connector_Molex:Molex_Micro-Fit_3.0_43650-0215_1x02_P3.00mm_Vertical
- J7: value PT_2 -> Conn_01x02; footprint Connector_JST:JST_XH_B2B-XH-A_1x02_P2.50mm_Vertical -> Connector_Molex:Molex_Micro-Fit_3.0_43650-0215_1x02_P3.00mm_Vertical
- J8: value PT_5 -> Conn_01x02; footprint Connector_JST:JST_XH_B2B-XH-A_1x02_P2.50mm_Vertical -> Connector_Molex:Molex_Micro-Fit_3.0_43650-0215_1x02_P3.00mm_Vertical
- J9: value PT_3 -> Conn_01x02; footprint Connector_JST:JST_XH_B2B-XH-A_1x02_P2.50mm_Vertical -> Connector_Molex:Molex_Micro-Fit_3.0_43650-0215_1x02_P3.00mm_Vertical
- moved J10 192.7 mm to (192.6, 82.6)
- moved J5 162.9 mm to (148.7, 33.2)
- moved R84 161.6 mm to (181.1, 81.7), turned to 180 degrees
- moved R82 159.1 mm to (181.7, 83.1)
- moved J14 158.9 mm to (192.6, 90.5)
- moved J15 158.9 mm to (192.6, 98.3)
- moved J16 158.9 mm to (192.6, 106.1)
- moved J17 158.9 mm to (192.6, 113.9)
- moved J18 158.9 mm to (192.6, 121.7)
- moved R88 154.3 mm to (181.2, 90.7), turned to 180 degrees
- moved J19 153.3 mm to (108.5, 41.1)
- moved R86 151.9 mm to (181.8, 92.1)
- moved R85 148.8 mm to (181.3, 108.7), turned to 180 degrees
- moved D32 147.9 mm to (185.4, 98.2), turned to 90 degrees
- moved R92 147.2 mm to (181.4, 99.7), turned to 180 degrees
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Connections:
- C55 pad 1: Net-(J5-Pin_1) -> Net-(J3-Pin_1)
- C56 pad 1: Net-(J6-Pin_1) -> Net-(J7-Pin_1)
- C57 pad 1: Net-(J7-Pin_1) -> Net-(J2-Pin_1)
- C59 pad 1: Net-(J9-Pin_1) -> Net-(J6-Pin_1)
- C60 pad 1: Net-(J10-Pin_1) -> Net-(J9-Pin_1)
- CR1 pad 1: Net-(CR1-Pad1) -> /ESP32 Breakout/D+
- CR1 pad 3: Net-(CR1-Pad3) -> /ESP32 Breakout/D-
- D17 pad 3: TC1+ -> /ThermocoupleADC1/AIN3
- D18 pad 3: TC1- -> /ThermocoupleADC1/AIN2
- D19 pad 3: TC2+ -> /ThermocoupleADC1/AIN1
- D20 pad 3: TC2- -> /ThermocoupleADC1/AIN0
- D21 pad 3: TC3+ -> /ThermocoupleADC2/AIN3
- D22 pad 3: TC3- -> /ThermocoupleADC2/AIN2
- D23 pad 3: TC4+ -> /ThermocoupleADC2/AIN1
- D24 pad 3: TC4- -> /ThermocoupleADC2/AIN0
- F1 pad 1: Net-(J2-POS) -> Net-(J19-Pin_1)
- F2 pad 1: /Ignitor Control/IGN_SUPPLY -> Net-(F2-Pad1)
- F2 pad 2: /Ignitor Control/IGNITOR_+VE -> /Ignitor Control/IGN_SUPPLY
- J10 pad 1: Net-(J10-Pin_1) -> +24V_SAFE
- J10 pad 2: PT_READ_6 -> /Valve Control/VALVE_1_RET
- J14 pad 2: /Valve Control/VALVE_1_RET -> /Valve Control/VALVE_2_RET
- J15 pad 2: /Valve Control/VALVE_4_RET -> /Valve Control/VALVE_3_RET
- J16 pad 1: +24V_SAFE -> +24V
- J16 pad 2: /Valve Control/VALVE_2_RET -> /Valve Control/VALVE_4_RET
- J18 pad 2: /Valve Control/VALVE_3_RET -> /Valve Control/VALVE_6_RET
- J19 pad 1: +24V -> Net-(J19-Pin_1)
- J19 pad 2: /Valve Control/VALVE_6_RET -> GND
- J2 pad 1: Net-(J2-POS) -> Net-(J2-Pin_1)
- J2 pad 2: GND -> PT_READ_2
- J3 pad 1: +24V -> Net-(J3-Pin_1)
- J3 pad 2: /Power Regulation/+24V_POST_LCKT -> PT_READ_1
- J5 pad 1: Net-(J5-Pin_1) -> /Power Regulation/+24V_POST_LCKT
- J5 pad 2: PT_READ_1 -> +24V
- J6 pad 2: PT_READ_4 -> PT_READ_3
- J7 pad 2: PT_READ_2 -> PT_READ_4
- J9 pad 2: PT_READ_3 -> PT_READ_6
- K2 pad 2: Net-(U12-+) -> Net-(K2-Pad2)
- K3 pad 2: /Ignitor Control/IGN_SUPPLY -> Net-(F2-Pad1)
- K3 pad 3: Net-(U12--) -> Net-(K2-Pad2)
- R64 pad 2: Net-(J5-Pin_1) -> Net-(J3-Pin_1)
- R65 pad 2: Net-(J6-Pin_1) -> Net-(J7-Pin_1)
- R68 pad 2: Net-(J7-Pin_1) -> Net-(J2-Pin_1)
- R72 pad 2: Net-(J9-Pin_1) -> Net-(J6-Pin_1)
- R73 pad 2: Net-(J10-Pin_1) -> Net-(J9-Pin_1)
- R77 pad 1: Net-(U12-+) -> /Ignitor Control/IGN_SUPPLY
- R77 pad 2: Net-(U12--) -> /Ignitor Control/IGNITOR_+VE
- U10 pad 1: +3.3V -> /ThermocoupleADC1/A0
- U10 pad 2: +3.3V -> /ThermocoupleADC1/A1
- U11 pad 1: I2C_SDA -> /ThermocoupleADC2/A0
- U11 pad 2: GND -> /ThermocoupleADC2/A1
- U12 pad 3: Net-(U12-+) -> /Ignitor Control/IGN_SUPPLY
- U12 pad 4: Net-(U12--) -> /Ignitor Control/IGNITOR_+VE
- U13 pad 1: GND -> /IgnitorADC/A0
- U13 pad 2: +3.3V -> /IgnitorADC/A1
- U8 pad 1: GND -> /ADC1/A0
- U8 pad 2: GND -> /ADC1/A1
- U9 pad 1: +3.3V -> /ADC2/A0
- U9 pad 2: GND -> /ADC2/A1
Routing:
- net GND: track 18.4 -> 126.3 mm, vias 16 -> 104
- net +24V: track 9.55 -> 96.0 mm, vias 0 -> 2
- net +24V_SAFE: track 0.00 -> 69.6 mm, vias 0 -> 1
- net +5V: track 0.00 -> 43.2 mm, vias 0 -> 30
- net /Power Regulation/+5.3V: track 30.1 -> 65.9 mm, vias 2 -> 4
- net /ThermocoupleADC1/AIN1: track 0.00 -> 25.2 mm
- net 5V_USB: track 1.44 -> 25.5 mm, vias 0 -> 3
- net +3.3V: track 2.67 -> 26.6 mm, vias 0 -> 11
- net /Power Regulation/+24V_POST_LCKT: track 0.00 -> 16.0 mm
- net Net-(K2-Pad2): track 0.00 -> 14.8 mm
- net /ESP32 Breakout/D+: track 0.00 -> 14.3 mm, vias 0 -> 2
- net /ThermocoupleADC2/AIN3: track 0.00 -> 13.5 mm
- net /ThermocoupleADC1/AIN3: track 0.00 -> 13.5 mm
- net /ThermocoupleADC1/AIN0: track 0.00 -> 13.4 mm
- net /ThermocoupleADC2/AIN0: track 0.00 -> 13.4 mm
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- added copper zone on F.Cu, net +24V
- added copper zone on F.Cu, net /Ignitor Control/IGN_SUPPLY
- added copper zone on B.Cu, net GND
Other:
- board size 122.9 x 136.7 mm -> 100 x 130 mm
