File: panda.kicad_pcb (KiCad board)
At the start: 4 copper layers, 100 x 130 mm, 266 parts, among them J1 Conn_01x02, J10 Conn_01x02, J11 4-Pin Load Cell, J12 5-Pin Load Cell, J13 Conn_02x01, J14 Conn_01x02, J15 Conn_01x02, J16 Conn_01x02, J17 Conn_01x02, J18 Conn_01x02, J19 Conn_01x02, J2 Conn_02x01, J20 395934308, J3 Conn_02x01, J4 USB_C_Receptacle_USB2.0_16P, J5 Conn_01x02, J6 Conn_01x02, J7 Conn_01x02, J8 Conn_01x02, J9 Conn_01x02, K1 G5Q-1A DC24, K2 G5Q-1 DC24, K3 G5Q-1 DC24, Q1 BSS138, Q10 BSS138, Q11 BSS138, Q2 BSS138, Q3 DMP6023LE-13, Q4 BSS138, Q5 BSS138, Q6 BSS138, Q7 BSS138, Q8 BSS138, Q9 BSS138, SW1 USAKRO UK-B0227-G4.3-B-250, SW2 USAKRO UK-B0227-G4.3-B-250, U1 LM3880-1AA, U10 ADS112C04, U11 ADS112C04, U12 INA187A1, U13 ADS112C04, U2 LMR33630BDDA, U3 TPS78533QKVURQ1, U4 TLC555xPS, U5 TPS78450QDBVRQ1, U6 LM66200DRLR, U7 ESP32-S3-WROOM-1U, U8 ADS112C04, U9 ADS112C04

Commit message: Resolve DRC issues
Parts:
- R45, R46, R47, R48, R54, R55, R56, R57: value Rb -> 1M
- moved Q2 1.23 mm to (115.0, 86.0)
Routing:
- net GND: track 209.0 -> 207.8 mm
- net Net-(Q2-G): track 22.3 -> 23.3 mm

Commit message: add silkscreen labels to connectors, remove pick Rb message (was already chosen)
Parts:
- moved BZ1 0.50 mm to (154.2, 65.2)
Other:
- board text added: "24VIN"
- board text added: "24V_SAFE_LOCK"
- board text added: "AV3"
- board text added: "AV4"
- board text added: "AV5"
- board text added: "AV6"
- board text added: "AV_FILL"
- board text added: "AV_RUN"
- board text added: "IGNITOR"
- board text added: "LC_FILL"
- board text added: "LC_THRUST"
- board text added: "PT1"
- board text added: "PT2"
- board text added: "PT3"
- board text added: "PT4"
- board text added: "PT5"
- board text added: "PT6"
- board text added: "PWR_ON_SW"
- board text added: "TC1- TC1+"
- board text added: "TC2- TC2+"
- board text added: "TC3- TC3+"
- board text added: "TC4- TC4+"
