File: IgnitorADC.kicad_sch (KiCad schematic)
At the start: 16 parts, among them U13 ADS112C04

Commit message: change clamping resistors on tc adcs for lower leakage current
Parts:
- renumbered R94 to R93, R95 to R94, R96 to R95, R97 to R96, R98 to R97
Changed lines of the file:
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@@
 		(on_board yes)
 		(dnp no)
-		(property "Reference" "R97"
+		(property "Reference" "R96"
 			(at 119.38 74.93 90)
 			(effects
@@
 			(project "panda"
 				(path "/226c5870-4123-4efa-a2b3-b42d02f59bb7/54d983a6-6da5-442c-8bd0-bcb1e102add1"
-					(reference "R97")
+					(reference "R96")
 					(unit 1)
 				)
@@
 		(on_board yes)
 		(dnp no)
-		(property "Reference" "#PWR0196"
+		(property "Reference" "#PWR0197"
 			(at 140.97 50.8 0)
 			(effects
@@
 			(project "panda"
 				(path "/226c5870-4123-4efa-a2b3-b42d02f59bb7/54d983a6-6da5-442c-8bd0-bcb1e102add1"
-					(reference "#PWR0196")
+					(reference "#PWR0197")
 					(unit 1)
 				)
@@
 		(on_board yes)
 		(dnp no)
-		(property "Reference" "#PWR0191"
+		(property "Reference" "#PWR0192"
 			(at 120.65 137.16 0)
 			(effects
@@
 			(project "panda"
 				(path "/226c5870-4123-4efa-a2b3-b42d02f59bb7/54d983a6-6da5-442c-8bd0-bcb1e102add1"
-					(reference "#PWR0191")
+					(reference "#PWR0192")
 					(unit 1)
 				)
@@
 		(on_board yes)
 		(dnp no)
-		(property "Reference" "#PWR0190"
+		(property "Reference" "#PWR0191"
 			(at 109.22 149.86 0)
 			(effects
@@
 			(project "panda"
 				(path "/226c5870-4123-4efa-a2b3-b42d02f59bb7/54d983a6-6da5-442c-8bd0-bcb1e102add1"
-					(reference "#PWR0190")
+					(reference "#PWR0191")
 					(unit 1)
 				)
@@
 		(on_board yes)
 		(dnp no)
-		(property "Reference" "#PWR0193"
+		(property "Reference" "#PWR0194"
 			(at 121.92 48.26 0)
 			(effects
@@
 			(project "panda"
 				(path "/226c5870-4123-4efa-a2b3-b42d02f59bb7/54d983a6-6da5-442c-8bd0-bcb1e102add1"
-					(reference "#PWR0193")
+					(reference "#PWR0194")
 					(unit 1)
 				)
@@
 		(on_board yes)
 		(dnp no)
-		(property "Reference" "#PWR0197"
+		(property "Reference" "#PWR0198"
 			(at 140.97 97.79 0)
 			(effects
@@
 			(project "panda"
 				(path "/226c5870-4123-4efa-a2b3-b42d02f59bb7/54d983a6-6da5-442c-8bd0-bcb1e102add1"
-					(reference "#PWR0197")
+					(reference "#PWR0198")
 					(unit 1)
 				)
@@
 		(on_board yes)
 		(dnp no)
-		(property "Reference" "R95"
+		(property "Reference" "R94"
 			(at 118.872 65.024 90)
 			(effects
@@
 			(project "panda"
 				(path "/226c5870-4123-4efa-a2b3-b42d02f59bb7/54d983a6-6da5-442c-8bd0-bcb1e102add1"
-					(reference "R95")
+					(reference "R94")
 					(unit 1)
 				)
@@
 		(on_board yes)
 		(dnp no)
-		(property "Reference" "#PWR0194"
+		(property "Reference" "#PWR0195"
 			(at 121.92 95.25 0)
 			(effects
@@
 			(project "panda"
 				(path "/226c5870-4123-4efa-a2b3-b42d02f59bb7/54d983a6-6da5-442c-8bd0-bcb1e102add1"
-					(reference "#PWR0194")
+					(reference "#PWR0195")
 					(unit 1)
 				)
@@
 		(on_board yes)
 		(dnp no)
-		(property "Reference" "R96"
+		(property "Reference" "R95"
 			(at 118.872 70.104 90)
 			(effects
@@
 			(project "panda"
 				(path "/226c5870-4123-4efa-a2b3-b42d02f59bb7/54d983a6-6da5-442c-8bd0-bcb1e102add1"
-					(reference "R96")
+					(reference "R95")
 					(unit 1)
 				)
@@
 		(on_board yes)
 		(dnp no)
-		(property "Reference" "R94"
+		(property "Reference" "R93"
 			(at 119.38 59.69 90)
 			(effects
@@
 			(project "panda"
 				(path "/226c5870-4123-4efa-a2b3-b42d02f59bb7/54d983a6-6da5-442c-8bd0-bcb1e102add1"
-					(reference "R94")
+					(reference "R93")
 					(unit 1)
 				)
@@
 		(on_board yes)
 		(dnp no)
-		(property "Reference" "#PWR0192"
+		(property "Reference" "#PWR0193"
 			(at 120.65 149.86 0)
 			(effects
@@
 			(project "panda"
 				(path "/226c5870-4123-4efa-a2b3-b42d02f59bb7/54d983a6-6da5-442c-8bd0-bcb1e102add1"
-					(reference "#PWR0192")
+					(reference "#PWR0193")
 					(unit 1)
 				)
@@
 		(on_board yes)
 		(dnp no)
-		(property "Reference" "#PWR0198"
+		(property "Reference" "#PWR0199"
 			(at 146.05 48.26 0)
 			(effects
@@
 			(project "panda"
 				(path "/226c5870-4123-4efa-a2b3-b42d02f59bb7/54d983a6-6da5-442c-8bd0-bcb1e102add1"
-					(reference "#PWR0198")
+					(reference "#PWR0199")
 					(unit 1)
 				)
@@
 		(on_board yes)
 		(dnp no)
-		(property "Reference" "#PWR0199"
+		(property "Reference" "#PWR0200"
 			(at 146.05 95.25 0)
 			(effects
@@
 			(project "panda"
 				(path "/226c5870-4123-4efa-a2b3-b42d02f59bb7/54d983a6-6da5-442c-8bd0-bcb1e102add1"
-					(reference "#PWR0199")
+					(reference "#PWR0200")
 					(unit 1)
 				)
@@
 		(on_board yes)
 		(dnp no)
-		(property "Reference" "#PWR0195"
+		(property "Reference" "#PWR0196"
 			(at 130.81 149.86 0)
 			(effects
@@
 			(project "panda"
 				(path "/226c5870-4123-4efa-a2b3-b42d02f59bb7/54d983a6-6da5-442c-8bd0-bcb1e102add1"
-					(reference "#PWR0195")
+					(reference "#PWR0196")
 					(unit 1)
 				)
@@
 		(on_board yes)
 		(dnp no)
-		(property "Reference" "#PWR0200"
+		(property "Reference" "#PWR0201"
 			(at 165.1 50.8 0)
 			(effects
@@
 			(project "panda"
 				(path "/226c5870-4123-4efa-a2b3-b42d02f59bb7/54d983a6-6da5-442c-8bd0-bcb1e102add1"
-					(reference "#PWR0200")
+					(reference "#PWR0201")
 					(unit 1)
 				)
@@
 		(on_board yes)
 		(dnp no)
-		(property "Reference" "R98"
+		(property "Reference" "R97"
 			(at 128.27 120.904 90)
 			(effects
@@
 			(project "panda"
 				(path "/226c5870-4123-4efa-a2b3-b42d02f59bb7/54d983a6-6da5-442c-8bd0-bcb1e102add1"
-					(reference "R98")
+					(reference "R97")
 					(unit 1)
 				)
@@
 		(on_board yes)
 		(dnp no)
-		(property "Reference" "#PWR0201"
+		(property "Reference" "#PWR0202"
 			(at 165.1 97.79 0)
 			(effects
@@
 			(project "panda"
 				(path "/226c5870-4123-4efa-a2b3-b42d02f59bb7/54d983a6-6da5-442c-8bd0-bcb1e102add1"
-					(reference "#PWR0201")
+					(reference "#PWR0202")
 					(unit 1)
 				)
@@
 		(on_board yes)
 		(dnp no)
-		(property "Reference" "#PWR0189"
+		(property "Reference" "#PWR0190"
 			(at 109.22 132.08 0)
 			(effects
@@
 			(project "panda"
 				(path "/226c5870-4123-4efa-a2b3-b42d02f59bb7/54d983a6-6da5-442c-8bd0-bcb1e102add1"
-					(reference "#PWR0189")
-					(unit 1)
-				)
+					(reference "#PWR0190")
+					(unit 1)
+				)

Commit message: Update version number in KiCad files
Other:
- company: (none) -> Queen's Rocket Engineering Team
- title: (none) -> PANDA
Changed lines of the file:
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@@
 	(generator_version "9.0")
 	(paper "A4")
+	(title_block
+		(title "PANDA")
+		(date "2025-12-21")
+		(rev "3.0.0")
+		(company "Queen's Rocket Engineering Team")
+	)
 	(rectangle
 		(start 102.87 106.68)
